File: SOT-363 to DIP/SOT-363 to DIP.kicad_sch (KiCad schematic)
At the start: 4 parts, among them J1 SOT-363, J2 Conn_01x03_Pin, J3 Conn_01x03_Pin, J4 SOT-353

Commit message: Remove silkscreen of pin headers
Parts:
- J2, J3: footprint Connector_PinHeader_2.54mm:PinHeader_1x03_P2.54mm_Vertical -> _footprints:PinHeader_1x03_P2.54mm_Vertical_nosilk
Changed lines of the file:
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@@
       (effects (font (size 1.27 1.27)) hide)
     )
-    (property "Footprint" "Connector_PinHeader_2.54mm:PinHeader_1x03_P2.54mm_Vertical" (at 35.56 110.49 0)
+    (property "Footprint" "_footprints:PinHeader_1x03_P2.54mm_Vertical_nosilk" (at 35.56 110.49 0)
       (effects (font (size 1.27 1.27)) hide)
     )
@@
       (effects (font (size 1.27 1.27)) (justify right) hide)
     )
-    (property "Footprint" "Connector_PinHeader_2.54mm:PinHeader_1x03_P2.54mm_Vertical" (at 59.69 110.49 0)
+    (property "Footprint" "_footprints:PinHeader_1x03_P2.54mm_Vertical_nosilk" (at 59.69 110.49 0)
       (effects (font (size 1.27 1.27)) hide)
     )
